Commit message: added world link/joint

File: water_maxi_description/urdf/water_maxi.urdf (robot description, URDF)
Before this commit: robot water_maxi, 2 links, 1 joints
Links:
- added link world
Joints:
- added joint world_to_Base: type fixed, parent world, child base_link, origin xyz=0 0 0 rpy=0 0 0, axis 0 0 0

Commit message: working on

File: water_maxi_description/urdf/water_maxi.urdf (robot description, URDF)
Before this commit: robot water_maxi, 3 links, 2 joints
Joints:
- removed joint base_to_arm
- added joint base_to_schwenkarm: type continuous, parent base_link, child arm_link1, origin xyz=-0.55 0 2 rpy=0.0 1.57 -1.57

Commit message: runs in Rviz

File: water_maxi_description/urdf/water_maxi.urdf (robot description, URDF)
Before this commit: robot water_maxi, 3 links, 2 joints
Joints:
- joint base_to_schwenkarm: axis (none) -> 0.0 1.0 0.0

Commit message: working on gazebo and ros_control

File: water_maxi_description/urdf/water_maxi.urdf (robot description, URDF)
Before this commit: robot water_maxi, 3 links, 2 joints
Links:
- link arm_link1: mass None -> 15.0; geometry collision mesh filename=package://water_maxi_description/models/SchwenkArm_Link.stl scale=0.01 0.01 0.01; visual mesh filename=package://water_maxi_description/models/SchwenkArm_Link.stl scale=0.01 0.01 0.01
- link base_link: mass None -> 1000.0; geometry collision mesh filename=package://water_maxi_description/models/Base_Link.stl scale=0.01 0.01 0.01; visual mesh filename=package://water_maxi_description/models/Base_Link.stl scale=0.01 0.01 0.01
Joints:
- joint world_to_Base: origin xyz=0 0 0 rpy=0 0 0 -> xyz=0 0 0.065 rpy=0 0 0

Commit message: gedanken spiel zum subscriber des füllstandwertes und publisher des Command wertes ungetestet

File: water_maxi_description/urdf/water_maxi.urdf (robot description, URDF)
Before this commit: robot water_maxi, 3 links, 2 joints
Joints:
- joint base_to_schwenkarm: axis 0.0 1.0 0.0 -> 0.0 -1.0 0.0
